File: hardware/gatormicrophone.brd (EAGLE design)
At the start: 38.1 x 38.1 mm, 81 parts, among them J1 GATORGATOR_MINI, J2 GATORGATOR_MINI, J3 GATORGATOR_MINI, J4 GATORGATOR_MINI, J5 GATORGATOR_MINI, J6 GATORGATOR_MINI, J7 GATORGATOR_MINI, J8 GATORGATOR_MINI, Q1 2.5A/30V/105mΩ, U1 ADS1015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

Commit message: engineer run of checklist
Parts:
- removed U$23: (no value), buzzard_labels (4):GATOR#SOUND1
- added U$24: (no value), buzzard_labels (15):GATOR#MICROPHONE0
- U$14: device buzzard_labels (4):GATOR#SOUND1 -> buzzard_labels (15):GATOR#MICROPHONE1
- moved LOGO3 21.9 mm to (8.26, 28.4)
- moved U$14 10.6 mm to (21.1, 25.4), flipped to the top
- moved R16 0.28 mm to (8.76, 9.78)
- turned D3 to 180 degrees
Routing:
- net SCL: track 56.6 -> 57.2 mm
Other:
- board text added: "v10"
- board text removed: "v01"
Changed lines of the file:
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@@
 <wire x1="38.1" y1="38.1" x2="0" y2="38.1" width="0.2032" layer="20"/>
 <text x="31.75" y="-10.16" size="1.778" layer="51" font="vector" ratio="10">Andy England</text>
-<text x="17.145" y="1.27" size="1.27" layer="16" font="vector" ratio="15" rot="MR0" align="center-right">v01</text>
+<text x="17.145" y="1.27" size="1.27" layer="16" font="vector" ratio="15" rot="MR0" align="center-right">v10</text>
 <wire x1="0" y1="38.1" x2="0" y2="24.13" width="0.2032" layer="20"/>
 <wire x1="0" y1="24.13" x2="2.54" y2="21.59" width="0.2032" layer="20"/>
@@
 <attribute name="VALUE" x="24.384" y="9.017" size="0.4064" layer="27" font="vector"/>
 </element>
-<element name="R16" library="SparkFun-Resistors" package="0603" value="1k" x="8.89" y="9.525" smashed="yes" rot="R180">
-<attribute name="NAME" x="9.779" y="8.763" size="0.4064" layer="25" font="vector" rot="R180"/>
-<attribute name="PROD_ID" value="RES-07856" x="8.89" y="9.525" size="1.778" layer="27" font="vector" ratio="15" rot="R180" display="off"/>
-<attribute name="VALUE" value="1k" x="9.906" y="10.668" size="0.4064" layer="27" font="vector" rot="R180"/>
-</element>
-<element name="D3" library="SparkFun-LED" package="LED-0603" value="RED" x="8.89" y="11.43" smashed="yes" rot="R90">
-<attribute name="NAME" x="9.779" y="10.7315" size="0.4064" layer="25" rot="R180"/>
-<attribute name="PROD_ID" value="DIO-00819" x="8.89" y="11.43" size="1.778" layer="27" font="vector" ratio="15" rot="R90" display="off"/>
-<attribute name="VALUE" x="9.906" y="12.5095" size="0.4064" layer="27" rot="R180"/>
+<element name="R16" library="SparkFun-Resistors" package="0603" value="1k" x="8.763" y="9.779" smashed="yes" rot="R180">
+<attribute name="NAME" x="9.652" y="9.017" size="0.4064" layer="25" font="vector" rot="R180"/>
+<attribute name="PROD_ID" value="RES-07856" x="8.763" y="9.779" size="1.778" layer="27" font="vector" ratio="15" rot="R180" display="off"/>
+<attribute name="VALUE" value="1k" x="9.779" y="10.922" size="0.4064" layer="27" font="vector" rot="R180"/>
+</element>
+<element name="D3" library="SparkFun-LED" package="LED-0603" value="RED" x="8.89" y="11.43" smashed="yes" rot="R180">
+<attribute name="NAME" x="9.5885" y="12.319" size="0.4064" layer="25" rot="R270"/>
+<attribute name="PROD_ID" value="DIO-00819" x="8.89" y="11.43" size="1.778" layer="27" font="vector" ratio="15" rot="R180" display="off"/>
+<attribute name="VALUE" x="7.8105" y="12.446" size="0.4064" layer="27" rot="R270"/>
 </element>
 <element name="LOGO1" library="SparkFun-Aesthetics" package="OSHW-LOGO-S" value="OSHW-LOGOS" x="19.05" y="3.175" smashed="yes" rot="MR0"/>
 <element name="LOGO2" library="SparkFun-Aesthetics" package="SFE_LOGO_NAME_FLAME_.2" value="SFE_LOGO_NAME_FLAME.2_INCH" x="18.796" y="17.78" smashed="yes" rot="MR0"/>
-<element name="LOGO3" library="SparkFun-Aesthetics" package="SFE_LOGO_FLAME_.2" value="SFE_LOGO_FLAME.2_INCH" x="29.845" y="24.638" smashed="yes"/>
+<element name="LOGO3" library="SparkFun-Aesthetics" package="SFE_LOGO_FLAME_.2" value="SFE_LOGO_FLAME.2_INCH" x="8.255" y="28.448" smashed="yes"/>
 <element name="C4" library="SparkFun-Capacitors" package="0603" value="1.0uF" x="8.89" y="16.51" smashed="yes">
 <attribute name="NAME" x="8.001" y="17.272" size="0.4064" layer="25" font="vector"/>
@@
 </element>
 <element name="U$21" library="buzzard_labels (8)" package="HIGH0" value="" x="1.27" y="24.765"/>
-<element name="U$14" library="buzzard_labels (4)" package="GATOR#SOUND1" value="" x="24.13" y="15.24" rot="MR0"/>
 <element name="TP1" library="SparkFun-Connectors" package="PAD.03X.03" value="TEST-POINT3" x="15.621" y="25.4" rot="MR0"/>
 <element name="H1" library="SparkFun-Hardware" package="STAND-OFF-TIGHT" value="STAND-OFFTIGHT" x="35.56" y="27.305" rot="R90"/>
@@
 </element>
 <element name="U$22" library="SparkFun-Aesthetics" package="ORDERING_INSTRUCTIONS" value="" x="-5.08" y="-15.24"/>
-<element name="U$23" library="buzzard_labels (4)" package="GATOR#SOUND1" value="" x="5.08" y="27.94"/>
+<element name="U$24" library="buzzard_labels (15)" package="GATOR#MICROPHONE0" value="" x="31.115" y="15.367" rot="MR0"/>
+<element name="U$14" library="buzzard_labels (15)" package="GATOR#MICROPHONE1" value="" x="21.082" y="25.4"/>
 </elements>
 <signals>
@@
 <via x="27.813" y="19.685" extent="1-16" drill="0.381"/>
 <via x="27.813" y="15.875" extent="1-16" drill="0.381"/>
-<via x="10.668" y="10.541" extent="1-16" drill="0.381"/>
+<via x="10.795" y="9.779" extent="1-16" drill="0.381"/>
 <via x="30.48" y="17.78" extent="1-16" drill="0.381"/>
 <via x="17.78" y="5.08" extent="1-16" drill="0.381"/>
@@
 <contactref element="D1" pad="C"/>
 <contactref element="R7" pad="2"/>
-<wire x1="17.565" y1="12.065" x2="15.24" y2="12.065" width="0.2032" layer="1"/>
-<wire x1="15.24" y1="11.365" x2="15.24" y2="12.065" width="0.2032" layer="1"/>
-<wire x1="18.2" y1="12.7" x2="17.565" y2="12.065" width="0.2032" layer="1"/>
-<wire x1="12.485" y1="13.97" x2="12.485" y2="12.407" width="0.2032" layer="1"/>
-<wire x1="12.485" y1="12.407" x2="12.827" y2="12.065" width="0.2032" layer="1"/>
-<wire x1="12.827" y1="12.065" x2="13.335" y2="12.065" width="0.2032" layer="1"/>
-<wire x1="13.335" y1="12.065" x2="15.24" y2="12.065" width="0.2032" layer="1"/>
-<wire x1="13.335" y1="11.365" x2="13.335" y2="12.065" width="0.2032" layer="1"/>
+<wire x1="12.485" y1="13.97" x2="12.485" y2="12.7" width="0.2032" layer="1"/>
+<wire x1="12.485" y1="12.7" x2="12.485" y2="11.645" width="0.2032" layer="1"/>
+<wire x1="12.765" y1="11.365" x2="13.335" y2="11.365" width="0.2032" layer="1"/>
+<wire x1="12.485" y1="11.645" x2="12.765" y2="11.365" width="0.2032" layer="1"/>
+<wire x1="13.335" y1="11.365" x2="15.24" y2="11.365" width="0.2032" layer="1"/>
+<wire x1="15.24" y1="11.365" x2="16.865" y2="11.365" width="0.2032" layer="1"/>
+<wire x1="16.865" y1="11.365" x2="18.2" y2="12.7" width="0.2032" layer="1"/>
 </signal>
 <signal name="N$10">
@@
 <contactref element="R16" pad="2"/>
 <contactref element="D3" pad="C"/>
-<wire x1="8.14" y1="11.43" x2="8.04" y2="11.33" width="0.2032" layer="1"/>
-<wire x1="8.04" y1="11.33" x2="8.04" y2="9.525" width="0.2032" layer="1"/>
+<wire x1="7.913" y1="11.33" x2="7.913" y2="9.779" width="0.2032" layer="1"/>
+<wire x1="8.013" y1="11.43" x2="7.913" y2="11.33" width="0.2032" layer="1"/>
 </signal>
 <signal name="ENVELOPE">
@@
 <wire x1="14.7125" y1="18.3075" x2="14.185" y2="17.78" width="0.1778" layer="1"/>
 <wire x1="10.287" y1="8.262" x2="11.43" y2="8.262" width="0.2032" layer="1"/>
-<wire x1="11.43" y1="8.262" x2="12.058" y2="8.262" width="0.2032" layer="1"/>
+<wire x1="11.684" y1="8.262" x2="12.058" y2="8.262" width="0.2032" layer="1"/>
 <wire x1="12.058" y1="8.262" x2="12.7" y2="7.62" width="0.2032" layer="1"/>
 <wire x1="12.7" y1="7.62" x2="18.2" y2="7.62" width="0.2032" layer="1"/>
-<wire x1="11.43" y1="8.262" x2="11.43" y2="11.43" width="0.2032" layer="1"/>
+<wire x1="11.557" y1="8.262" x2="11.557" y2="11.43" width="0.2032" layer="1"/>
 <via x="11.43" y="14.859" extent="1-16" drill="0.381"/>
-<wire x1="11.43" y1="11.43" x2="11.43" y2="14.859" width="0.2032" layer="1"/>
+<wire x1="11.557" y1="11.43" x2="11.557" y2="14.732" width="0.2032" layer="1"/>
 <wire x1="11.43" y1="14.859" x2="11.43" y2="16.891" width="0.2032" layer="16"/>
 <via x="11.43" y="16.891" extent="1-16" drill="0.381"/>
 <wire x1="11.43" y1="16.891" x2="13.296" y2="16.891" width="0.2032" layer="1"/>
 <wire x1="13.296" y1="16.891" x2="14.185" y2="17.78" width="0.2032" layer="1"/>
-<wire x1="9.64" y1="11.43" x2="11.43" y2="11.43" width="0.2032" layer="1"/>
 <wire x1="18.2" y1="19.47" x2="18.2" y2="20.32" width="0.2032" layer="1"/>
 <wire x1="18.2" y1="20.32" x2="18.2" y2="23.114" width="0.2032" layer="1"/>
@@
 <wire x1="16.25" y1="18.415" x2="14.82" y2="18.415" width="0.2032" layer="1"/>
 <wire x1="14.82" y1="18.415" x2="14.7125" y2="18.3075" width="0.2032" layer="1"/>
+<wire x1="11.557" y1="8.262" x2="11.684" y2="8.262" width="0.2032" layer="1"/>
+<wire x1="9.767" y1="11.43" x2="11.43" y2="11.43" width="0.2032" layer="1"/>
+<wire x1="11.557" y1="14.732" x2="11.43" y2="14.859" width="0.2032" layer="1"/>
+<wire x1="11.43" y1="11.43" x2="11.557" y2="11.43" width="0.2032" layer="1"/>
+<wire x1="11.43" y1="8.262" x2="11.557" y2="8.262" width="0.2032" layer="1"/>
 </signal>
 <signal name="N$13">
@@
 <wire x1="29.21" y1="4.699" x2="31.242" y2="6.731" width="0.2032" layer="1"/>
 <wire x1="31.242" y1="6.731" x2="31.242" y2="7.62" width="0.2032" layer="1"/>
-<wire x1="33.02" y1="24.13" x2="33.02" y2="30.21" width="0.2032" layer="1"/>
-<wire x1="36.83" y1="20.32" x2="33.02" y2="24.13" width="0.2032" layer="1"/>
+<wire x1="31.75" y1="25.4" x2="31.75" y2="30.21" width="0.2032" layer="1"/>
+<wire x1="36.83" y1="20.32" x2="31.75" y2="25.4" width="0.2032" layer="1"/>
 <wire x1="33.02" y1="30.21" x2="33.893" y2="30.21" width="0.2032" layer="1"/>
 <wire x1="33.893" y1="30.21" x2="34.29" y2="30.607" width="0.2032" layer="1"/>
@@
 <wire x1="22.082" y1="27.67" x2="22.606" y2="28.194" width="0.2032" layer="1"/>
 <wire x1="22.606" y1="28.194" x2="24.622" y2="30.21" width="0.2032" layer="1"/>
-<wire x1="24.622" y1="30.21" x2="33.02" y2="30.21" width="0.2032" layer="1"/>
+<wire x1="31.75" y1="30.21" x2="33.02" y2="30.21" width="0.2032" layer="1"/>
+<wire x1="24.622" y1="30.21" x2="31.75" y2="30.21" width="0.2032" layer="1"/>
 </signal>
 <signal name="N$19">
