File: hardware/gatormicrophone.sch (EAGLE design)
At the start: 58 parts, among them J1 GATORGATOR_MINI, J2 GATORGATOR_MINI, J3 GATORGATOR_MINI, J4 GATORGATOR_MINI, J5 GATORGATOR_MINI, J6 GATORGATOR_MINI, J7 GATORGATOR_MINI, J8 GATORGATOR_MINI, Q1 2.5A/30V/105mΩ, U1 ADS1015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

Commit message: engineer run of checklist
Other:
- note added: "7-bit Unshifted I2CAddress: 0x48"
- note added: "Supply Voltage: 2.7-3.6V."
- note added: "v10"
- note removed: "Address: 0x48"
- note removed: "Vcc range between 2.7V and 3.6V."
- note removed: "v01"
- moved on the sheet: R19
Changed lines of the file:
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@@
 <plain>
 <text x="165.608" y="11.43" size="2.54" layer="94" font="vector">Andrew England</text>
-<text x="238.76" y="7.62" size="2.54" layer="94" font="vector">v01</text>
+<text x="238.76" y="7.62" size="2.54" layer="94" font="vector">v10</text>
 <wire x1="0" y1="104.14" x2="60.96" y2="104.14" width="0.1524" layer="97" style="longdash"/>
 <wire x1="60.96" y1="104.14" x2="114.3" y2="104.14" width="0.1524" layer="97" style="longdash"/>
@@
 <text x="124.46" y="99.06" size="2.54" layer="97" font="vector">Schmitt trigger</text>
 <text x="116.84" y="167.64" size="1.778" layer="97" font="vector">Half-wave precision rectifier with gain of approx 2</text>
-<text x="2.54" y="96.52" size="1.778" layer="97" font="vector">Vcc range between 2.7V and 3.6V.</text>
+<text x="2.54" y="96.52" size="1.778" layer="97" font="vector">Supply Voltage: 2.7-3.6V.</text>
 <wire x1="121.92" y1="53.34" x2="121.92" y2="104.14" width="0.1524" layer="97" style="longdash"/>
 <wire x1="0" y1="53.34" x2="121.92" y2="53.34" width="0.1524" layer="97" style="longdash"/>
 <text x="2.54" y="48.26" size="2.54" layer="97" font="vector">ADC-to-I2C</text>
-<text x="73.66" y="7.62" size="1.778" layer="97" font="vector">Address: 0x48</text>
+<text x="20.32" y="7.62" size="1.778" layer="97" font="vector">7-bit Unshifted I2CAddress: 0x48</text>
 </plain>
 <instances>
@@
 <attribute name="VALUE" x="222.25" y="116.078" size="1.778" layer="96" font="vector"/>
 </instance>
-<instance part="R19" gate="G$1" x="96.52" y="119.38" smashed="yes">
-<attribute name="NAME" x="92.71" y="120.8786" size="1.778" layer="95" font="vector"/>
-<attribute name="VALUE" x="92.71" y="116.078" size="1.778" layer="96" font="vector"/>
+<instance part="R19" gate="G$1" x="91.44" y="121.92" smashed="yes" rot="R270">
+<attribute name="NAME" x="92.9386" y="125.73" size="1.778" layer="95" font="vector" rot="R270"/>
+<attribute name="VALUE" x="88.138" y="125.73" size="1.778" layer="96" font="vector" rot="R270"/>
 </instance>
 <instance part="FID3" gate="G$1" x="218.44" y="27.94" smashed="yes"/>
@@
 </instance>
 <instance part="C5" gate="G$1" x="15.24" y="25.4"/>
-<instance part="TP1" gate="G$1" x="38.1" y="27.94" rot="R180"/>
+<instance part="TP1" gate="G$1" x="38.1" y="27.94" smashed="yes" rot="R180">
+<attribute name="NAME" x="40.64" y="27.432" size="1.778" layer="95" font="vector" rot="R180"/>
+</instance>
 <instance part="H1" gate="G$1" x="223.52" y="30.48"/>
 <instance part="H2" gate="G$1" x="223.52" y="27.94"/>
@@
 <segment>
 <pinref part="R19" gate="G$1" pin="2"/>
-<wire x1="101.6" y1="119.38" x2="104.14" y2="119.38" width="0.1524" layer="91"/>
-<label x="104.14" y="119.38" size="1.27" layer="95" font="vector" xref="yes"/>
+<wire x1="91.44" y1="116.84" x2="91.44" y2="114.3" width="0.1524" layer="91"/>
+<label x="91.44" y="114.3" size="1.27" layer="95" font="vector" rot="R270" xref="yes"/>
 </segment>
 <segment>
@@
 <pinref part="C4" gate="G$1" pin="1"/>
 <pinref part="R19" gate="G$1" pin="1"/>
-<wire x1="91.44" y1="129.54" x2="91.44" y2="119.38" width="0.1524" layer="91"/>
+<wire x1="91.44" y1="129.54" x2="91.44" y2="127" width="0.1524" layer="91"/>
 <pinref part="S1" gate="G$1" pin="3"/>
 <wire x1="99.06" y1="157.48" x2="96.52" y2="157.48" width="0.1524" layer="91"/>
